File: sapphire_radio_esp32.kicad_pcb (KiCad board)
At the start: 2 copper layers, 160 x 95 mm, 129 parts, among them IC1 AZ1117CH-3.3TRG1, J1 GT-USB-7055E, J2 Screw_Terminal_01x02, J3 FAKRA, J4 Screw_Terminal_01x02, J5 Screw_Terminal_01x02, Q1 DMG2305UX-7, Q2 DMP3013SFV-7, Q3 2N7002PS_115, SW1 1825027-8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

Commit message: Add board first pass; move ESP32 GPIO to allow easier routing
Parts:
- removed C30: 10uF, Capacitor_SMD:CP_Elec_4x5.4
- added D4: LED, Connector_JST:JST_ZH_B2B-ZR-SM4-TF_1x02-1MP_P1.50mm_Vertical, F.Cu at (173.2, 105.2)
- added J6: Conn_01x03, Connector_JST:JST_PH_B3B-PH-SM4-TB_1x03-1MP_P2.00mm_Vertical, F.Cu at (55.9, 94.7)
- added R38: 5, Resistor_SMD:R_0603_1608Metric, F.Cu at (170.0, 107.2)
- R34: value 10k -> 100k
- moved FB5 214.8 mm to (143.8, 117.1)
- moved FB7 211.5 mm to (139.0, 128.2), turned to 90 degrees
- moved FB6 210.4 mm to (140.6, 113.7)
- moved C9 208.7 mm to (160.7, 110.4), turned to -90 degrees
- moved FB4 206.2 mm to (135.7, 110.8)
- moved FB3 203.0 mm to (131.4, 112.5), turned to 90 degrees
- moved C38 200.4 mm to (156.1, 110.4), turned to -90 degrees
- moved C42 193.9 mm to (139.0, 124.9), turned to -90 degrees
- moved C37 191.0 mm to (142.4, 119.1)
- moved C47 186.9 mm to (141.2, 116.1), turned to -90 degrees
- moved C50 186.1 mm to (143.5, 115.4), turned to 180 degrees
- moved C41 184.9 mm to (135.0, 128.8)
- moved C40 184.1 mm to (134.1, 126.5), turned to -90 degrees
- moved C49 183.8 mm to (141.6, 111.3), turned to 90 degrees
- moved C46 183.7 mm to (139.0, 110.7)
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Connections:
- R22 pad 2: /~{MUTE} -> Net-(U5-A1)
- U1 pad 10: /B5 -> /ESP32_I2S_CLK
- U1 pad 11: unconnected-(U1-IO26-Pad11) -> /SI4735_SDIO
- U1 pad 12: /DAC_GAIN -> /SI4735_SCLK
- U1 pad 13: /DAC_FILTER -> /~{SI_EN}
- U1 pad 15: unconnected-(U1-GND-Pad15) -> GND
- U1 pad 16: /~{MUTE} -> /ESP32_I2S_DOUT
- U1 pad 23: /SI4735_SCLK -> /DAC_GAIN
- U1 pad 24: /SI4735_SDIO -> /MUX_SEL
- U1 pad 25: /~{SI_EN} -> /DAC_FILTER
- U1 pad 26: unconnected-(U1-IO4-Pad26) -> /DIAL_SERVO
- U1 pad 27: unconnected-(U1-IO16-Pad27) -> /B1
- U1 pad 28: /ESP32_I2S_DFS -> /B2
- U1 pad 29: /ESP32_I2S_DOUT -> /B3
- U1 pad 30: /MUX_SEL -> /B4
- U1 pad 31: /ESP32_I2S_CLK -> /B5
- U1 pad 33: unconnected-(U1-IO21-Pad33) -> /I2C_BUS_SDA
- U1 pad 37: /I2C_BUS_SDA -> unconnected-(U1-IO23-Pad37)
- U1 pad 5: unconnected-(U1-SENSOR_VN-Pad5) -> /SEEK
- U1 pad 6: /B1 -> unconnected-(U1-IO34-Pad6)
- U1 pad 7: /B2 -> unconnected-(U1-IO35-Pad7)
- U1 pad 8: /B3 -> /ESP32_I2S_DFS
- U1 pad 9: /B4 -> VCC
- U5 pad 1: /~{MUTE} -> Net-(U5-A1)
- U8 pad 9: /I2C_BUS_SCLK -> /I2C_BUS_SCL
Routing:
- net VCC: track 65.4 -> 525.2 mm, vias 0 -> 27
- net /VOLUME: track 0.00 -> 306.0 mm, vias 0 -> 4
- net +BATT: track 0.00 -> 269.5 mm, vias 0 -> 2
- net GND: track 9.31 -> 132.8 mm, vias 0 -> 74
- net /I2C_BUS_SCL: track 0.00 -> 118.8 mm, vias 0 -> 4
- net /B1: track 0.00 -> 112.8 mm
- net /I2C_BUS_SDA: track 0.00 -> 111.4 mm, vias 0 -> 2
- net /B2: track 0.00 -> 94.4 mm
- net /~{RESET}: track 56.2 -> 143.7 mm, vias 2 -> 10
- net /B3: track 0.00 -> 80.1 mm
- net /MUTE: track 0.00 -> 70.5 mm, vias 0 -> 4
- net /B4: track 0.00 -> 62.9 mm
- net /ESP32_I2S_DFS: track 3.21 -> 63.8 mm, vias 1 -> 2
- net Net-(C52-Pad1): track 0.00 -> 57.6 mm
- net /ESP32_I2S_CLK: track 14.1 -> 69.1 mm, vias 0 -> 4
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- added copper zone on B.Cu, net GND
- added copper zone on F.Cu, net GND

Commit message: Final WROOM revision
Parts:
- removed U2: CP2102N-A02-GQFN24R, carter_kicad_footprints:QFN50P400X400X80-25N
- added C30: 0.47uF, Capacitor_SMD:C_0603_1608Metric, F.Cu at (49.8, 118.6)
- added IC2: AS169-73LF, carter_kicad_footprints:SOT95P270X145-6N, F.Cu at (48.4, 107.2)
- added IC3: CP2102N-A02-GQFN28R, carter_kicad_footprints:QFN50P700X700X80-45N, F.Cu at (59.5, 51.5)
- added R39: 10k, Resistor_SMD:R_0603_1608Metric, F.Cu at (47.0, 104.6)
- added R40: 10k, Resistor_SMD:R_0603_1608Metric, F.Cu at (46.7, 91.0)
- added R41: 10k, Resistor_SMD:R_0603_1608Metric, F.Cu at (62.2, 66.2)
- added U3: NC7WZ14P6X, carter_kicad_footprints:SC70-6_ONS, F.Cu at (47.6, 93.7)
- moved R8 12.1 mm to (50.3, 59.5), turned to 180 degrees
- moved R1 11.4 mm to (49.0, 48.8)
- moved R5 10.8 mm to (53.5, 49.6), turned to 180 degrees
- moved S1 9.57 mm to (44.0, 58.8)
- moved C6 6.66 mm to (51.6, 53.4)
- moved C7 6.59 mm to (53.1, 53.4)
- moved R12 6.58 mm to (59.3, 59.6), turned to 0 degrees
- moved Q3 6.17 mm to (56.0, 59.5), turned to 180 degrees
- moved R4 4.07 mm to (49.8, 57.6)
- moved J1 3.89 mm to (44.2, 51.8), turned to 90 degrees
- moved C5 3.76 mm to (52.8, 57.5), turned to 180 degrees
- moved D3 3.70 mm to (49.0, 54.2)
- moved R3 3.18 mm to (56.3, 56.4), turned to 180 degrees
- moved C1 2.69 mm to (43.9, 104.4), turned to 180 degrees
- moved R2 2.30 mm to (40.5, 53.2), turned to -90 degrees
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Connections:
- C22 pad 1: Net-(J3-SIGNAL) -> /FMI
- C22 pad 2: /FMI -> Net-(U4-FMI)
- J3 pad 1: Net-(J3-SIGNAL) -> Net-(IC2-J1)
- L2 pad 1: /FMI -> Net-(U4-FMI)
- U1 pad 37: unconnected-(U1-IO23-Pad37) -> /FM_SEL
- U4 pad 12: unconnected-(U4-AMI-Pad12) -> Net-(U4-AMI)
- U4 pad 8: /FMI -> Net-(U4-FMI)
- U4 pad 9: unconnected-(U4-RFGND-Pad9) -> GND
- UD2 pad 2: Net-(J3-SIGNAL) -> Net-(IC2-J1)
Routing:
- net /FM_SEL: track 0.00 -> 61.2 mm, vias 0 -> 4
- net VCC: track 525.2 -> 546.8 mm, vias 27 -> 31
- net GND: track 132.8 -> 153.6 mm, vias 74 -> 119
- net /~{RESET}: track 143.7 -> 126.4 mm
- net /AM_SEL: track 0.00 -> 16.6 mm, vias 0 -> 2
- net /AM: track 0.00 -> 12.9 mm
- net Net-(J3-SIGNAL): track 12.2 -> 0.00 mm
- net VBUS: track 64.6 -> 75.4 mm
- net Net-(IC2-J1): track 0.00 -> 9.73 mm
- net /RTS: track 7.39 -> 16.0 mm
- net /DTR: track 16.8 -> 23.0 mm, vias 4 -> 2
- net /DP: track 23.9 -> 17.9 mm, vias 4 -> 2
- net /FMI: track 3.40 -> 8.56 mm
- net /UART_TX: track 30.1 -> 25.0 mm
- net /UART_RX: track 27.9 -> 23.2 mm
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
Commit message: Move fakra to board edge; move associated parts; silkscreen
Parts:
- added G***: LOGO, carter_kicad_footprints:cjh_cone_18mm, F.Cu at (190.9, 93.8)
- moved UD2 13.8 mm to (43.7, 121.8)
- moved J3 13.6 mm to (43.8, 128.2)
- moved IC2 10.9 mm to (46.5, 117.9), turned to -90 degrees
- moved R39 8.18 mm to (43.3, 111.9), turned to 90 degrees
- moved R5 8.15 mm to (55.9, 57.4), turned to 0 degrees
- moved R3 2.60 mm to (58.9, 56.4), turned to 0 degrees
- moved U3 0.60 mm to (47.0, 93.7)
Connections:
- R22 pad 1: VCC -> GND
- R22 pad 2: Net-(U5-A1) -> /MUTE
- U1 pad 9: VCC -> /MUTE
- U5 pad 1: Net-(U5-A1) -> /MUTE
- U5 pad 6: /MUTE -> /~{MUTE}
Routing:
- net /MUTE: track 70.5 -> 152.0 mm, vias 4 -> 14
- net GND: track 153.6 -> 191.1 mm, vias 119 -> 186
- net /~{MUTE}: track 0.00 -> 23.5 mm, vias 0 -> 2
- net /FM_SEL: track 61.2 -> 73.6 mm, vias 4 -> 6
- net /AM_SEL: track 16.6 -> 28.8 mm
- net /VOLUME: track 307.4 -> 319.4 mm, vias 4 -> 6
- net /AM: track 12.9 -> 5.24 mm
- net /FMI: track 8.56 -> 2.49 mm
- net Net-(IC3-RSTB): track 4.43 -> 8.74 mm, vias 0 -> 2
- net Net-(IC3-VBUS): track 14.9 -> 12.5 mm, vias 3 -> 2
- net Net-(U6-~{EN}): track 5.27 -> 2.94 mm
- net VCC: track 546.8 -> 544.5 mm
- net Net-(U5-A1): track 1.80 -> 0.00 mm
- net Net-(IC3-VDD): track 12.7 -> 13.6 mm
- net /SI4735_SCLK: track 45.6 -> 45.0 mm
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Other:
- board text added: "+"
- board text added: "-"
- board text added: "DIAL SERVO SIG + -"
- board text added: "Designed by Carter Harris - KE8OHO"
- board text added: "L SPKR"
- board text added: "MAIN POWER"
- board text added: "PH"
- board text added: "PWR LED"
- board text added: "R SPKR"
- board text added: "TO RADIO ANTENNA FAKRA CONN"
- board text added: "TUNE"
- board text added: "VOLUME & POWER"
- board text added: "VW Sapphire XVIII v1.0 Radio Conversion Apr 26 AM/FM/Bluetooth"
- board text added: "ZH"
